File: Hardware_Design/KiCad_Schematics/relay_control_circuit/relay_control_circuit.kicad_pcb (KiCad board)
At the start: 2 copper layers, 6 parts, among them J1 Screw_Terminal_01x02, K2 SANYOU_SRD_Form_C, SW1 SW_Push

Commit message: Add README and clean up schematic for Relay Control Circuit
Added the README.md file for the Relay Control Circuit project. Refactored the schematic and PCB layout to be cleaner and more visually appealing by reducing unnecessary screw terminals into a single block, simplifying the overall design.
Routing:
- added copper zone on B.Cu, net GND
Changed lines of the file:
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@@
 (kicad_pcb
-	(version 20241229)
+	(version 20260206)
 	(generator "pcbnew")
-	(generator_version "9.0")
+	(generator_version "10.0")
 	(general
 		(thickness 1.6)
@@
 		(pad_to_mask_clearance 0)
 		(allow_soldermask_bridges_in_footprints no)
-		(tenting front back)
+		(tenting
+			(front yes)
+			(back yes)
+		)
+		(covering
+			(front no)
+			(back no)
+		)
+		(plugging
+			(front no)
+			(back no)
+		)
+		(capping no)
+		(filling no)
 		(pcbplotparams
 			(layerselection 0x00000000_00000000_55555555_5755f5ff)
@@
 			(usegerberadvancedattributes yes)
 			(creategerberjobfile yes)
-			(dashed_line_dash_ratio 12.000000)
-			(dashed_line_gap_ratio 3.000000)
+			(dashed_line_dash_ratio 12)
+			(dashed_line_gap_ratio 3)
 			(svgprecision 4)
 			(plotframeref no)
 			(mode 1)
 			(useauxorigin no)
-			(hpglpennumber 1)
-			(hpglpenspeed 20)
-			(hpglpendiameter 15.000000)
 			(pdf_front_fp_property_popups yes)
 			(pdf_back_fp_property_popups yes)
@@
 		)
 	)
-	(net 0 "")
-	(net 1 "Net-(D1-K)")
-	(net 2 "GND")
-	(net 3 "Net-(D2-A)")
-	(net 4 "+12V")
-	(net 5 "Net-(K2-Pad3)")
-	(net 6 "unconnected-(K2-Pad4)")
 	(footprint "LED_THT:LED_D5.0mm"
 		(layer "F.Cu")
@@
 		(sheetfile "kurs2.kicad_sch")
 		(attr through_hole)
+		(duplicate_pad_numbers_are_jumpers no)
 		(fp_line
 			(start -1.29 -1.545)
@@
 			(layers "*.Cu" "*.Mask")
 			(remove_unused_layers no)
-			(net 2 "GND")
+			(net "GND")
 			(pinfunction "K")
 			(pintype "passive")
@@
 			(layers "*.Cu" "*.Mask")
 			(remove_unused_layers no)
-			(net 3 "Net-(D2-A)")
+			(net "Net-(D2-A)")
 			(pinfunction "A")
 			(pintype "passive")
@@
 		(sheetfile "kurs2.kicad_sch")
 		(attr through_hole)
+		(duplicate_pad_numbers_are_jumpers no)
 		(fp_line
 			(start 1.34 0)
@@
 			(remove_unused_layers no)
 			(roundrect_rratio 0.113636)
-			(net 1 "Net-(D1-K)")
+			(net "Net-(D1-K)")
 			(pinfunction "K")
 			(pintype "passive")
@@
 			(layers "*.Cu" "*.Mask")
 			(remove_unused_layers no)
-			(net 2 "GND")
+			(net "GND")
 			(pinfunction "A")
 			(pintype "passive")
@@
 		(sheetfile "kurs2.kicad_sch")
 		(attr through_hole)
+		(duplicate_pad_numbers_are_jumpers no)
 		(fp_line
 			(start 6.75 3)
@@
 			(layers "*.Cu" "*.Mask")
 			(remove_unused_layers no)
-			(net 1 "Net-(D1-K)")
+			(net "Net-(D1-K)")
 			(pinfunction "1")
 			(pintype "passive")
@@
 			(layers "*.Cu" "*.Mask")
 			(remove_unused_layers no)
-			(net 1 "Net-(D1-K)")
+			(net "Net-(D1-K)")
 			(pinfunction "1")
 			(pintype "passive")
@@
 			(layers "*.Cu" "*.Mask")
 			(remove_unused_layers no)
-			(net 4 "+12V")
+			(net "+12V")
 			(pinfunction "2")
 			(pintype "passive")
@@
 			(layers "*.Cu" "*.Mask")
 			(remove_unused_layers no)
-			(net 4 "+12V")
+			(net "+12V")
 			(pinfunction "2")
 			(pintype "passive")
@@
 		(sheetfile "kurs2.kicad_sch")
 		(attr through_hole)
+		(duplicate_pad_numbers_are_jumpers no)
 		(fp_line
 			(start -2.66 -5.32)
@@
 			(remove_unused_layers no)
 			(roundrect_rratio 0.096154)
-			(net 4 "+12V")
+			(net "+12V")
 			(pinfunction "Pin_1")
 			(pintype "passive")
@@
 			(layers "*.Cu" "*.Mask")
 			(remove_unused_layers no)
-			(net 2 "GND")
+			(net "GND")
 			(pinfunction "Pin_2")
 			(pintype "passive")
@@
 		(sheetfile "kurs2.kicad_sch")
 		(attr through_hole)
+		(duplicate_pad_numbers_are_jumpers no)
 		(fp_line
 			(start -1.4 -7.8)
@@
 			(layers "*.Cu" "*.Mask")
 			(remove_unused_layers no)
-			(net 4 "+12V")
+			(net "+12V")
 			(pintype "passive")
 		)
@@
 			(layers "*.Cu" "*.Mask")
 			(remove_unused_layers no)
-			(net 2 "GND")
+			(net "GND")
 			(pintype "passive")
 		)
@@
 			(layers "*.Cu" "*.Mask")
 			(remove_unused_layers no)
-			(net 5 "Net-(K2-Pad3)")
+			(net "Net-(K2-Pad3)")
 			(pintype "passive")
 		)
@@
 			(layers "*.Cu" "*.Mask")
 			(remove_unused_layers no)
-			(net 6 "unconnected-(K2-Pad4)")
+			(net "unconnected-(K2-Pad4)")
 			(pintype "passive+no_connect")
 		)
@@
 			(layers "*.Cu" "*.Mask")
 			(remove_unused_layers no)
-			(net 1 "Net-(D1-K)")
+			(net "Net-(D1-K)")
 			(pintype "passive")
 		)
@@
 		(sheetfile "kurs2.kicad_sch")
 		(attr through_hole)
+		(duplicate_pad_numbers_are_jumpers no)
 		(fp_line
 			(start 9.12 0)
@@
 			(layers "*.Cu" "*.Mask")
 			(remove_unused_layers no)
-			(net 5 "Net-(K2-Pad3)")
+			(net "Net-(K2-Pad3)")
 			(pintype "passive")
 		)
@@
 			(layers "*.Cu" "*.Mask")
 			(remove_unused_layers no)
-			(net 3 "Net-(D2-A)")
+			(net "Net-(D2-A)")
 			(pintype "passive")
 		)
@@
 		(width 0.2)
 		(layer "F.Cu")
-		(net 1)
+		(net "Net-(D1-K)")
 	)
 	(segment
@@
 		(width 0.2)
 		(layer "F.Cu")
-		(net 1)
+		(net "Net-(D1-K)")
 	)
 	(segment
@@
 		(width 0.2)
 		(layer "F.Cu")
-		(net 1)
+		(net "Net-(D1-K)")
 	)
 	(segment
@@
 		(width 0.2)
 		(layer "F.Cu")
-		(net 1)
+		(net "Net-(D1-K)")
 	)
 	(segment
@@
 		(width 0.2)
 		(layer "F.Cu")
-		(net 1)
+		(net "Net-(D1-K)")
 	)
 	(segment
@@
 		(width 0.2)
 		(layer "F.Cu")
-		(net 1)
+		(net "Net-(D1-K)")
 	)
 	(segment
@@
 		(width 0.2)
 		(layer "F.Cu")
-		(net 2)
+		(net "GND")
 	)
 	(segment
@@
 		(width 0.2)
 		(layer "F.Cu")
-		(net 2)
+		(net "GND")
 	)
 	(segment
@@
 		(width 0.2)
 		(layer "F.Cu")
-		(net 2)
+		(net "GND")
 	)
 	(segment
@@
 		(width 0.2)
 		(layer "F.Cu")
-		(net 2)
+		(net "GND")
 	)
 	(segment
@@
 		(width 0.2)
 		(layer "F.Cu")
-		(net 2)
+		(net "GND")
 	)
 	(segment
@@
 		(width 0.2)
 		(layer "F.Cu")
-		(net 2)
+		(net "GND")
 	)
 	(segment
@@
 		(width 0.2)
 		(layer "F.Cu")
-		(net 2)
+		(net "GND")
 	)
 	(segment
@@
 		(width 0.2)
 		(layer "F.Cu")
-		(net 2)
+		(net "GND")
 	)
 	(segment
@@
 		(width 0.2)
 		(layer "F.Cu")
-		(net 3)
+		(net "Net-(D2-A)")
 	)
 	(segment
@@
 		(width 0.2)
 		(layer "F.Cu")
-		(net 3)
+		(net "Net-(D2-A)")
 	)
 	(segment
@@
 		(width 0.2)
 		(layer "F.Cu")
-		(net 4)
+		(net "+12V")
 	)
 	(segment
@@
 		(width 0.2)
 		(layer "F.Cu")
-		(net 4)
+		(net "+12V")
 	)
 	(segment
@@
 		(width 0.2)
 		(layer "F.Cu")
-		(net 4)
+		(net "+12V")
 	)
 	(segment
@@
 		(width 0.2)
 		(layer "F.Cu")
-		(net 4)
+		(net "+12V")
 	)
 	(segment
@@
 		(width 0.2)
 		(layer "F.Cu")
-		(net 4)
+		(net "+12V")
 	)
 	(segment
@@
 		(width 0.2)
 		(layer "F.Cu")
-		(net 5)
+		(net "Net-(K2-Pad3)")
 	)
 	(segment
@@
 		(width 0.2)
 		(layer "F.Cu")
-		(net 5)
+		(net "Net-(K2-Pad3)")
+	)
+	(zone
+		(net "GND")
+		(layer "B.Cu")
+		(hatch edge 0.5)
+		(connect_pads
+			(clearance 0.5)
+		)
+		(min_thickness 0.25)
+		(fill yes
+			(thermal_gap 0.5)
+			(thermal_bridge_width 0.5)
+			(island_removal_mode 0)
+		)
+		(polygon
+			(pts
+				(xy 139.5 87) (xy 179.5 87) (xy 180 119.5) (xy 139.5 119)
+			)
+		)
 	)
 	(embedded_fonts no)
