File: Hardware_Design/KiCad_Schematics/Buck Converter/buck_hierarchical.kicad_sch (KiCad schematic)
At the start: 6 parts, among them Q1 2N7002

Commit message: Update designs but continue problems...
Added a Bootstrap circuit to bring the MOSFET from a Linear Regulator state to a Buck Converter state, but the problem is still not resolved. While it should yield a value close to 6V when the Duty Cycle is at 50% and a 12V input is applied, it yields 4V, and the graph is not correct. Work on the problem will continue.
Connections:
- net SOURCE: now reaches D1.1 (K), L1.1, Q1.2 (S)
- net PULSE renamed GATE
Other:
- moved on the sheet: C1, C2, D1, L1, Q1, R1
Changed lines of the file:
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@@
 	)
 	(junction
-		(at 146.05 86.36)
+		(at 146.05 87.63)
 		(diameter 0)
 		(color 0 0 0 0)
 	)
 	(junction
-		(at 137.16 86.36)
+		(at 137.16 87.63)
 		(diameter 0)
 		(color 0 0 0 0)
 	)
 	(junction
-		(at 129.54 86.36)
+		(at 129.54 87.63)
 		(diameter 0)
 		(color 0 0 0 0)
@@
 	(wire
 		(pts
-			(xy 147.32 86.36) (xy 146.05 86.36)
+			(xy 147.32 87.63) (xy 146.05 87.63)
 		)
 		(stroke
@@
 	(wire
 		(pts
-			(xy 146.05 86.36) (xy 137.16 86.36)
+			(xy 146.05 87.63) (xy 137.16 87.63)
 		)
 		(stroke
@@
 	(hierarchical_label "GND"
 		(shape passive)
-		(at 129.54 93.98 270)
+		(at 129.54 95.25 270)
 		(effects
 			(font
@@
 	(hierarchical_label "OUTPUT"
 		(shape output)
-		(at 147.32 86.36 0)
+		(at 147.32 87.63 0)
 		(effects
 			(font
@@
 			)
 			(justify left)
+		)
+	)
+	(hierarchical_label "GATE"
+		(shape input)
+		(at 124.46 95.25 270)
+		(effects
+			(font
+				(size 1.27 1.27)
+			)
+			(justify right)
 		)
 	)
 	(hierarchical_label "DC"
 		(shape input)
-		(at 119.38 86.36 180)
+		(at 119.38 87.63 180)
 		(effects
 			(font
@@
 	(hierarchical_label "GND"
 		(shape passive)
-		(at 119.38 93.98 270)
+		(at 119.38 95.25 270)
 		(effects
 			(font
@@
 	(hierarchical_label "GND"
 		(shape passive)
-		(at 137.16 93.98 270)
-		(effects
-			(font
-				(size 1.27 1.27)
-			)
-			(justify right)
-		)
-	)
-	(hierarchical_label "PULSE"
-		(shape input)
-		(at 124.46 93.98 270)
+		(at 137.16 95.25 270)
 		(effects
 			(font
@@
 	(hierarchical_label "GND"
 		(shape passive)
-		(at 146.05 93.98 270)
+		(at 146.05 95.25 270)
 		(effects
 			(font
@@
 			)
 			(justify right)
+		)
+	)
+	(hierarchical_label "SOURCE"
+		(shape input)
+		(at 129.54 87.63 90)
+		(effects
+			(font
+				(size 1.27 1.27)
+			)
+			(justify left)
 		)
 	)
 	(symbol
 		(lib_id "Device:R")
-		(at 146.05 90.17 0)
+		(at 146.05 91.44 0)
 		(unit 1)
 		(body_style 1)
@@
 		(fields_autoplaced yes)
 		(property "Reference" "R1"
-			(at 148.59 88.8999 0)
+			(at 148.59 90.1699 0)
 			(show_name no)
 			(do_not_autoplace no)
@@
 		)
 		(property "Value" "1k"
-			(at 148.59 91.4399 0)
+			(at 148.59 92.7099 0)
 			(show_name no)
 			(do_not_autoplace no)
@@
 		)
 		(property "Footprint" "Resistor_THT:R_Axial_DIN0204_L3.6mm_D1.6mm_P5.08mm_Horizontal"
-			(at 144.272 90.17 90)
+			(at 144.272 91.44 90)
 			(hide yes)
 			(show_name no)
@@
 		)
 		(property "Datasheet" ""
-			(at 146.05 90.17 0)
+			(at 146.05 91.44 0)
 			(hide yes)
 			(show_name no)
@@
 		)
 		(property "Description" "Resistor"
-			(at 146.05 90.17 0)
+			(at 146.05 91.44 0)
 			(hide yes)
 			(show_name no)
@@
 	(symbol
 		(lib_id "Device:C")
-		(at 137.16 90.17 0)
+		(at 137.16 91.44 0)
 		(unit 1)
 		(body_style 1)
@@
 		(dnp no)
 		(property "Reference" "C2"
-			(at 139.446 89.154 0)
+			(at 139.446 90.424 0)
 			(show_name no)
 			(do_not_autoplace no)
@@
 		)
 		(property "Value" "100u"
-			(at 139.446 91.186 0)
+			(at 139.446 92.456 0)
 			(show_name no)
 			(do_not_autoplace no)
@@
 		)
 		(property "Footprint" "Capacitor_THT:CP_Radial_D4.0mm_P1.50mm"
-			(at 138.1252 93.98 0)
+			(at 138.1252 95.25 0)
 			(hide yes)
 			(show_name no)
@@
 		)
 		(property "Datasheet" ""
-			(at 137.16 90.17 0)
+			(at 137.16 91.44 0)
 			(hide yes)
 			(show_name no)
@@
 		)
 		(property "Description" "Unpolarized capacitor"
-			(at 137.16 90.17 0)
+			(at 137.16 91.44 0)
 			(hide yes)
 			(show_name no)
@@
 	(symbol
 		(lib_id "Device:L")
-		(at 133.35 86.36 90)
+		(at 133.35 87.63 90)
 		(unit 1)
 		(body_style 1)
@@
 		(dnp no)
 		(property "Reference" "L1"
-			(at 133.096 83.058 90)
+			(at 133.096 84.328 90)
 			(show_name no)
 			(do_not_autoplace no)
@@
 		)
 		(property "Value" "100u"
-			(at 133.096 84.836 90)
+			(at 133.096 86.106 90)
 			(show_name no)
 			(do_not_autoplace no)
@@
 		)
 		(property "Footprint" "Inductor_THT:L_Radial_D6.0mm_P4.00mm"
-			(at 133.35 86.36 0)
+			(at 133.35 87.63 0)
 			(hide yes)
 			(show_name no)
@@
 		)
 		(property "Datasheet" ""
-			(at 133.35 86.36 0)
+			(at 133.35 87.63 0)
 			(hide yes)
 			(show_name no)
@@
 		)
 		(property "Description" "Inductor"
-			(at 133.35 86.36 0)
+			(at 133.35 87.63 0)
 			(hide yes)
 			(show_name no)
@@
 	(symbol
 		(lib_id "Device:D_Schottky")
-		(at 129.54 90.17 270)
+		(at 129.54 91.44 270)
 		(unit 1)
 		(body_style 1)
@@
 		(dnp no)
 		(property "Reference" "D1"
-			(at 131.064 89.154 90)
+			(at 131.064 90.424 90)
 			(show_name no)
 			(do_not_autoplace no)
@@
 		)
 		(property "Value" "0.3"
-			(at 131.064 91.186 90)
+			(at 131.064 92.456 90)
 			(show_name no)
 			(do_not_autoplace no)
@@
 		)
 		(property "Footprint" "Diode_THT:D_A-405_P7.62mm_Horizontal"
-			(at 129.54 90.17 0)
+			(at 129.54 91.44 0)
 			(hide yes)
 			(show_name no)
@@
 		)
 		(property "Datasheet" ""
-			(at 129.54 90.17 0)
+			(at 129.54 91.44 0)
 			(hide yes)
 			(show_name no)
@@
 		)
 		(property "Description" "Schottky diode"
-			(at 129.54 90.17 0)
+			(at 129.54 91.44 0)
 			(hide yes)
 			(show_name no)
@@
 	(symbol
 		(lib_id "Transistor_FET:2N7002")
-		(at 124.46 88.9 90)
+		(at 124.46 90.17 90)
 		(unit 1)
 		(body_style 1)
@@
 		(fields_autoplaced yes)
 		(property "Reference" "Q1"
-			(at 124.46 80.01 90)
+			(at 124.46 81.28 90)
 			(show_name no)
 			(do_not_autoplace no)
@@
 		)
 		(property "Value" "2N7002"
-			(at 124.46 82.55 90)
+			(at 124.46 83.82 90)
 			(show_name no)
 			(do_not_autoplace no)
@@
 		)
 		(property "Footprint" "Package_TO_SOT_THT:TO-220-3_Vertical"
-			(at 126.365 83.82 0)
+			(at 126.365 85.09 0)
 			(hide yes)
 			(show_name no)
@@
 		)
 		(property "Datasheet" "https://www.onsemi.com/pub/Collateral/NDS7002A-D.PDF"
-			(at 128.27 83.82 0)
+			(at 128.27 85.09 0)
 			(hide yes)
 			(show_name no)
@@
 		)
 		(property "Description" "0.115A Id, 60V Vds, N-Channel MOSFET, SOT-23"
-			(at 124.46 88.9 0)
+			(at 124.46 90.17 0)
 			(hide yes)
 			(show_name no)
@@
 	(symbol
 		(lib_id "Device:C")
-		(at 119.38 90.17 0)
+		(at 119.38 91.44 0)
 		(unit 1)
 		(body_style 1)
@@
 		(dnp no)
 		(property "Reference" "C1"
-			(at 114.046 88.9 0)
+			(at 114.046 90.17 0)
 			(show_name no)
 			(do_not_autoplace no)
@@
 		)
 		(property "Value" "100u"
-			(at 114.046 91.44 0)
+			(at 114.046 92.71 0)
 			(show_name no)
 			(do_not_autoplace no)
@@
 		)
 		(property "Footprint" "Capacitor_THT:CP_Radial_D4.0mm_P1.50mm"
-			(at 120.3452 93.98 0)
+			(at 120.3452 95.25 0)
 			(hide yes)
 			(show_name no)
@@
 		)
 		(property "Datasheet" ""
-			(at 119.38 90.17 0)
+			(at 119.38 91.44 0)
 			(hide yes)
 			(show_name no)
@@
 		)
 		(property "Description" "Unpolarized capacitor"
-			(at 119.38 90.17 0)
-			(hide yes)
-			(show_name no)
+			(at 119.38 91.44 0)
+			(hide yes)
+			(show_name no)
