File: Hardware_Design/KiCad_Schematics/Buck Converter/bootstrap_driver.kicad_sch (KiCad schematic)
At the start: 0 parts

Commit message: Update designs but continue problems...
Added a Bootstrap circuit to bring the MOSFET from a Linear Regulator state to a Buck Converter state, but the problem is still not resolved. While it should yield a value close to 6V when the Duty Cycle is at 50% and a 12V input is applied, it yields 4V, and the graph is not correct. Work on the problem will continue.
Parts:
- added C_BOOT1: 1u, symbol Device:C
- added D_BOOT1: D_Schotky, symbol Device:D_Schottky
- added Q3: PNP, symbol Simulation_SPICE:PNP
- added Q4: NPN, symbol Simulation_SPICE:NPN
- added R_BASE1: 100, symbol Device:R
- added R_GATE1: 10, symbol Device:R
Connections:
- new net: Q3.2 (B), Q4.2 (B), R_BASE1.1
- new net: Q3.3 (E), Q4.3 (E), R_GATE1.2
- new net SIMBOOT: C_BOOT1.2, D_BOOT1.1 (K), Q4.1 (C)
- new net SIMGATE: R_GATE1.1
- new net SIMPULSE: R_BASE1.2
- new net SIMSOURCE: C_BOOT1.1, Q3.1 (C)
- new net SIMVCC: D_BOOT1.2 (A)
