File: Hardware_Design/KiCad_Schematics/kicad-custom-symbols-learning/kicad-custom-symbols-learning/kicad-custom-symbols-learning.kicad_sch (KiCad schematic)
At the start: 0 parts

Commit message: feat(custom-symbols-learning): add custom LM386 symbol design
Parts:
- added U1: (no value), symbol Display_Character:Custom-LM386
Changed lines of the file:
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@@
 	(generator_version "10.0")
 	(paper "A4")
+	(symbol
+		(lib_id "Display_Character:Custom-LM386")
+		(at 144.78 105.41 0)
+		(unit 1)
+		(body_style 1)
+		(exclude_from_sim no)
+		(in_bom yes)
+		(on_board yes)
+		(in_pos_files yes)
+		(dnp no)
+		(fields_autoplaced yes)
+		(property "Reference" "U1"
+			(at 144.78 97.79 0)
+			(show_name no)
+			(do_not_autoplace no)
+			(effects
+				(font
+					(size 1.27 1.27)
+				)
+			)
+		)
+		(property "Value" ""
+			(at 144.78 105.41 0)
+			(show_name no)
+			(do_not_autoplace no)
+			(effects
+				(font
+					(size 1.27 1.27)
+				)
+			)
+		)
+		(property "Footprint" ""
+			(at 144.78 105.41 0)
+			(hide yes)
+			(show_name no)
+			(do_not_autoplace no)
+			(effects
+				(font
+					(size 1.27 1.27)
+				)
+			)
+		)
+		(property "Datasheet" ""
+			(at 144.78 105.41 0)
+			(hide yes)
+			(show_name no)
+			(do_not_autoplace no)
+			(effects
+				(font
+					(size 1.27 1.27)
+				)
+			)
+		)
+		(property "Description" ""
+			(at 144.78 105.41 0)
+			(hide yes)
+			(show_name no)
+			(do_not_autoplace no)
+			(effects
+				(font
+					(size 1.27 1.27)
+				)
+			)
+		)
+		(pin "2"
+		)
+		(pin "3"
+		)
+		(pin "4"
+		)
+		(pin "1"
+		)
+		(pin "6"
+		)
+		(pin "7"
+		)
+		(pin "5"
+		)
+		(pin "8"
+		)
+		(instances
+			(project "kicad-custom-symbols-learning"
+				(path "/f018fdee-1270-4361-a55e-f2d02016429b"
+					(reference "U1")
+					(unit 1)
+				)
+			)
+		)
+	)
 	(sheet_instances
 		(path "/"

Commit message: resize and simplify LM386 symbol design
fix design because it was very small, complex and unreadable.
Parts:
- removed U1: (no value), symbol Display_Character:Custom-LM386
Changed lines of the file:
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@@
 	(generator_version "10.0")
 	(paper "A4")
-	(symbol
-		(lib_id "Display_Character:Custom-LM386")
-		(at 144.78 105.41 0)
-		(unit 1)
-		(body_style 1)
-		(exclude_from_sim no)
-		(in_bom yes)
-		(on_board yes)
-		(in_pos_files yes)
-		(dnp no)
-		(fields_autoplaced yes)
-		(property "Reference" "U1"
-			(at 144.78 97.79 0)
-			(show_name no)
-			(do_not_autoplace no)
-			(effects
-				(font
-					(size 1.27 1.27)
-				)
-			)
-		)
-		(property "Value" ""
-			(at 144.78 105.41 0)
-			(show_name no)
-			(do_not_autoplace no)
-			(effects
-				(font
-					(size 1.27 1.27)
-				)
-			)
-		)
-		(property "Footprint" ""
-			(at 144.78 105.41 0)
-			(hide yes)
-			(show_name no)
-			(do_not_autoplace no)
-			(effects
-				(font
-					(size 1.27 1.27)
-				)
-			)
-		)
-		(property "Datasheet" ""
-			(at 144.78 105.41 0)
-			(hide yes)
-			(show_name no)
-			(do_not_autoplace no)
-			(effects
-				(font
-					(size 1.27 1.27)
-				)
-			)
-		)
-		(property "Description" ""
-			(at 144.78 105.41 0)
-			(hide yes)
-			(show_name no)
-			(do_not_autoplace no)
-			(effects
-				(font
-					(size 1.27 1.27)
-				)
-			)
-		)
-		(pin "2"
-		)
-		(pin "3"
-		)
-		(pin "4"
-		)
-		(pin "1"
-		)
-		(pin "6"
-		)
-		(pin "7"
-		)
-		(pin "5"
-		)
-		(pin "8"
-		)
-		(instances
-			(project "kicad-custom-symbols-learning"
-				(path "/f018fdee-1270-4361-a55e-f2d02016429b"
-					(reference "U1")
-					(unit 1)
-				)
-			)
-		)
-	)
 	(sheet_instances
 		(path "/"

Commit message: feat(custom-symbols-learning): add typical LM386 application circuit example
Parts:
- added C2, C5: C, symbol Device:C
- added C3: 0.05uF, symbol Device:C
- added C4: 250uF, symbol Device:C
- added J1: Conn_01x03_Socket, Connector_PinSocket_1.00mm:PinSocket_1x03_P1.00mm_Vertical, symbol Connector:Conn_01x03_Socket
- added LS1: Speaker, symbol Device:Speaker
- added R1: 10k, symbol Device:R
- added R2: 10, symbol Device:R
- added U1: (no value), symbol Display_Character:Custom-LM386
Connections:
- new net: C3.2, R2.1
- new net: C4.2, LS1.1
- new net: C5.1, U1.1
- new net: C5.2, U1.8
- new net: R1.2, U1.3
- new net: C2.1, U1.7
- new net: C3.1, C4.1, U1.5
- new net AUDIO-IN: J1.1 (Pin_1), R1.1
- new net GND: C2.2, J1.3 (Pin_3), LS1.2, R2.2, U1.2, U1.4
- new net Vs: J1.2 (Pin_2), U1.6

Commit message: feat(custom-symbols-learning): add footprints
Parts:
- C2, C3, C4, C5: footprint (none) -> Capacitor_THT:CP_Radial_D5.0mm_P2.50mm
- LS1: footprint (none) -> Buzzer_Beeper:Speaker_CUI_CMR-1206S-67
- R1, R2: footprint (none) -> Resistor_THT:R_Axial_DIN0207_L6.3mm_D2.5mm_P15.24mm_Horizontal
- U1: footprint (none) -> Package_DIP:DIP-8_W7.62mm
Changed lines of the file:
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@@
 			)
 		)
-		(property "Footprint" ""
+		(property "Footprint" "Resistor_THT:R_Axial_DIN0207_L6.3mm_D2.5mm_P15.24mm_Horizontal"
 			(at 140.462 116.84 90)
 			(hide yes)
@@
 			)
 		)
-		(property "Footprint" ""
+		(property "Footprint" "Buzzer_Beeper:Speaker_CUI_CMR-1206S-67"
 			(at 158.75 110.49 0)
 			(hide yes)
@@
 			)
 		)
-		(property "Footprint" ""
+		(property "Footprint" "Capacitor_THT:CP_Radial_D5.0mm_P2.50mm"
 			(at 143.51 87.9348 0)
 			(hide yes)
@@
 			)
 		)
-		(property "Footprint" ""
+		(property "Footprint" "Resistor_THT:R_Axial_DIN0207_L6.3mm_D2.5mm_P15.24mm_Horizontal"
 			(at 130.81 104.648 90)
 			(hide yes)
@@
 			)
 		)
-		(property "Footprint" ""
+		(property "Footprint" "Capacitor_THT:CP_Radial_D5.0mm_P2.50mm"
 			(at 149.86 99.3648 0)
 			(hide yes)
@@
 			)
 		)
-		(property "Footprint" ""
+		(property "Footprint" "Package_DIP:DIP-8_W7.62mm"
 			(at 139.7 101.6 0)
 			(hide yes)
@@
 			)
 		)
-		(property "Footprint" ""
+		(property "Footprint" "Capacitor_THT:CP_Radial_D5.0mm_P2.50mm"
 			(at 149.86 104.4448 0)
 			(hide yes)
@@
 			)
 		)
-		(property "Footprint" ""
+		(property "Footprint" "Capacitor_THT:CP_Radial_D5.0mm_P2.50mm"
 			(at 143.2052 113.03 0)
 			(hide yes)
